File: BizBopWhingWhang/LEDSheet.kicad_sch (KiCad schematic)
At the start: 111 parts, among them U10 74HC595, U11 74HC595, U12 74HC595, U5 74HC595, U6 74HC595, U7 74HC595

Commit message: Latest version
Parts:
- U10, U11, U12, U5, U6, U7: footprint Package_SO:TSSOP-16-1EP_4.4x5mm_P0.65mm -> Package_SO:TSSOP-16_4.4x5mm_P0.65mm
Changed lines of the file:
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@@
       (effects (font (size 1.27 1.27)) (justify left))
     )
-    (property "Footprint" "Package_SO:TSSOP-16-1EP_4.4x5mm_P0.65mm" (id 2) (at 225.425 40.64 0)
+    (property "Footprint" "Package_SO:TSSOP-16_4.4x5mm_P0.65mm" (id 2) (at 225.425 40.64 0)
       (effects (font (size 1.27 1.27)) hide)
     )
@@
   (symbol (lib_id "74xx:74HC595") (at 147.32 135.255 0) (unit 1)
     (in_bom yes) (on_board yes) (fields_autoplaced)
-    (property "Reference" "U10" (id 0) (at 149.3394 117.475 0)
-      (effects (font (size 1.27 1.27)) (justify left))
-    )
-    (property "Value" "74HC595" (id 1) (at 149.3394 120.015 0)
-      (effects (font (size 1.27 1.27)) (justify left))
-    )
-    (property "Footprint" "Package_SO:TSSOP-16-1EP_4.4x5mm_P0.65mm" (id 2) (at 147.32 135.255 0)
+    (property "Reference" "U10" (id 0) (at 149.3394 116.84 0)
+      (effects (font (size 1.27 1.27)) (justify left))
+    )
+    (property "Value" "74HC595" (id 1) (at 149.3394 119.38 0)
+      (effects (font (size 1.27 1.27)) (justify left))
+    )
+    (property "Footprint" "Package_SO:TSSOP-16_4.4x5mm_P0.65mm" (id 2) (at 147.32 135.255 0)
       (effects (font (size 1.27 1.27)) hide)
     )
@@
       (effects (font (size 1.27 1.27)) (justify left))
     )
-    (property "Footprint" "Package_SO:TSSOP-16-1EP_4.4x5mm_P0.65mm" (id 2) (at 64.77 90.17 0)
+    (property "Footprint" "Package_SO:TSSOP-16_4.4x5mm_P0.65mm" (id 2) (at 64.77 90.17 0)
       (effects (font (size 1.27 1.27)) hide)
     )
@@
       (effects (font (size 1.27 1.27)) (justify left))
     )
-    (property "Footprint" "Package_SO:TSSOP-16-1EP_4.4x5mm_P0.65mm" (id 2) (at 226.06 87.63 0)
+    (property "Footprint" "Package_SO:TSSOP-16_4.4x5mm_P0.65mm" (id 2) (at 226.06 87.63 0)
       (effects (font (size 1.27 1.27)) hide)
     )
@@
   (symbol (lib_id "74xx:74HC595") (at 64.77 42.545 0) (unit 1)
     (in_bom yes) (on_board yes) (fields_autoplaced)
-    (property "Reference" "U5" (id 0) (at 66.7894 24.765 0)
-      (effects (font (size 1.27 1.27)) (justify left))
-    )
-    (property "Value" "74HC595" (id 1) (at 66.7894 27.305 0)
-      (effects (font (size 1.27 1.27)) (justify left))
-    )
-    (property "Footprint" "Package_SO:TSSOP-16-1EP_4.4x5mm_P0.65mm" (id 2) (at 64.77 42.545 0)
+    (property "Reference" "U5" (id 0) (at 66.7894 24.13 0)
+      (effects (font (size 1.27 1.27)) (justify left))
+    )
+    (property "Value" "74HC595" (id 1) (at 66.7894 26.67 0)
+      (effects (font (size 1.27 1.27)) (justify left))
+    )
+    (property "Footprint" "Package_SO:TSSOP-16_4.4x5mm_P0.65mm" (id 2) (at 64.77 42.545 0)
       (effects (font (size 1.27 1.27)) hide)
     )
@@
       (effects (font (size 1.27 1.27)) (justify left))
     )
-    (property "Footprint" "Package_SO:TSSOP-16-1EP_4.4x5mm_P0.65mm" (id 2) (at 64.77 137.16 0)
-      (effects (font (size 1.27 1.27)) hide)
-    )
+    (property "Footprint" "Package_SO:TSSOP-16_4.4x5mm_P0.65mm" (id 2) (at 64.77 137.16 0)
+      (effects (font (size 1.27 1.27)) hide)
+    )
