File: BizBopWhingWhang/BizBopWhingWhang.kicad_pcb (KiCad board)
At the start: 2 copper layers, 40 x 55 mm, 148 parts, among them J1 USB_C_Receptacle_USB2.0-Conne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, J3 Conn_01x03, SW1 SW_Push, SW2 SW_Push, U1 AMS1117-3.3, U10 74HC595, U11 74HC595, U12 74HC595, U2 W25Q128JVSIQ, U3 RP2040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

Commit message: Latest version
Parts:
- removed SW1, SW2: SW_Push, BizBopWhingWhang:K2-1808UN
- removed U4: 74HC245, Package_SO:TSSOP-20_4.4x6.5mm_P0.65mm
- added D49: D_Photo, BizBopWhingWhang:PD-1522CTR8, F.Cu at (145.4, 113.8)
- added JP1: Bridge, Connector_PinHeader_2.54mm:PinHeader_1x02_P2.54mm_Vertical, F.Cu at (163.4, 102.4)
- added JP2: Bridge, Connector_PinHeader_2.54mm:PinHeader_1x02_P2.54mm_Vertical, F.Cu at (137.5, 98.4)
- added R58: 100k, Resistor_SMD:R_0603_1608Metric_Pad0.98x0.95mm_HandSolder, F.Cu at (154.1, 114.1)
- U10, U11, U12, U5, U6, U7: footprint Package_SO:TSSOP-16-1EP_4.4x5mm_P0.65mm -> Package_SO:TSSOP-16_4.4x5mm_P0.65mm
- moved R9 14.8 mm to (140.2, 98.5), turned to 90 degrees
- moved C14 6.05 mm to (139.7, 104.3)
- moved J3 5.84 mm to (156.2, 109.4)
- moved R57 5.51 mm to (134.1, 102.0), turned to -90 degrees
- moved R24 3.02 mm to (141.1, 116.2), turned to -90 degrees
- moved R44 2.49 mm to (158.6, 109.2)
- moved R52 2.43 mm to (158.1, 117.9)
- moved R55 2.38 mm to (161.3, 121.9)
- moved R54 2.33 mm to (160.2, 121.9)
- moved R56 2.30 mm to (162.5, 121.9)
- moved R50 2.30 mm to (156.8, 117.8)
- moved R53 2.27 mm to (159.1, 121.8)
- moved R41 2.20 mm to (160.1, 99.8), turned to 180 degrees
- moved R40 2.19 mm to (162.5, 132.4)
- moved C17 2.15 mm to (152.0, 111.6), turned to 180 degrees
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Connections:
- U10 pad 11: SCK -> GPIO2
- U10 pad 12: RCLK -> GPIO8
- U10 pad 13: OE -> GPIO10
- U11 pad 11: SCK -> GPIO2
- U11 pad 12: RCLK -> GPIO8
- U11 pad 13: OE -> GPIO10
- U12 pad 11: SCK -> GPIO2
- U12 pad 12: RCLK -> GPIO8
- U12 pad 13: OE -> GPIO10
- U5 pad 11: SCK -> GPIO2
- U5 pad 12: RCLK -> GPIO8
- U5 pad 13: OE -> GPIO10
- U6 pad 11: SCK -> GPIO2
- U6 pad 12: RCLK -> GPIO8
- U6 pad 13: OE -> GPIO10
- U7 pad 11: SCK -> GPIO2
- U7 pad 12: RCLK -> GPIO8
- U7 pad 13: OE -> GPIO10
Routing:
- net OE: track 118.7 -> 0.00 mm
- net RCLK: track 118.6 -> 0.00 mm, vias 10 -> 0
- net GPIO10: track 13.5 -> 130.1 mm
- net SCK: track 116.1 -> 0.00 mm, vias 10 -> 0
- net GPIO8: track 12.7 -> 124.2 mm, vias 0 -> 12
- net GPIO2: track 11.3 -> 117.4 mm, vias 0 -> 12
- net GPIO26: track 0.00 -> 23.3 mm, vias 0 -> 2
- net QSPISS: track 16.2 -> 7.77 mm, vias 4 -> 0
- net +3.3V: track 372.2 -> 376.7 mm, vias 23 -> 22
- net Net-(J3-Pad3): track 8.78 -> 12.2 mm
- net Net-(D16-Pad1): track 4.53 -> 7.23 mm
- net Net-(D48-Pad1): track 15.7 -> 13.2 mm
- net Net-(J3-Pad1): track 10.7 -> 8.19 mm
- net Net-(D47-Pad1): track 14.0 -> 11.6 mm
- net Net-(JP2-Pad1): track 5.37 -> 3.00 mm
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
Commit message: Added first draft of code
Parts:
- R5: footprint Resistor_SMD:R_0603_1608Metric_Pad0.98x0.95mm_HandSolder -> Resistor_SMD:R_0402_1005Metric
- moved C17 3.93 mm to (155.5, 113.4)
- moved C16 3.48 mm to (149.5, 111.7), turned to 0 degrees
- moved D49 2.72 mm to (147.9, 115.0), turned to 0 degrees
- moved R58 2.60 mm to (155.7, 112.1), turned to 180 degrees
- moved Y1 1.68 mm to (152.2, 113.4), turned to -90 degrees
- moved C7 0.86 mm to (150.4, 110.4), turned to 0 degrees
- moved R5 0.52 mm to (148.0, 111.9)
- moved C9 0.34 mm to (148.5, 110.4), turned to 180 degrees
Routing:
- net +3.3V: track 376.7 -> 381.3 mm
- net Net-(C17-Pad2): track 6.22 -> 8.83 mm
- net GND: track 60.7 -> 58.6 mm, vias 52 -> 53
- net GPIO26: track 23.3 -> 21.8 mm
- net Net-(R5-Pad2): track 2.25 -> 2.78 mm
