File: BizBopWhingWhang/BizBopWhingWhang.kicad_sch (KiCad schematic)
At the start: 37 parts, among them J1 USB_C_Receptacle_USB2.0-Conne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, J3 Conn_01x03, SW1 SW_Push, SW2 SW_Push, U1 AMS1117-3.3, U2 W25Q128JVSIQ, U3 RP2040, U4 74HC245, Y1 12 MHz

Commit message: Latest version
Parts:
- removed SW1, SW2: SW_Push, BizBopWhingWhang:K2-1808UN, symbol Switch:SW_Push
- removed U4: 74HC245, Package_SO:TSSOP-20_4.4x6.5mm_P0.65mm, symbol 74xx:74HC245
- added D49: D_Photo, BizBopWhingWhang:PD-1522CTR8, symbol Device:D_Photo
- added JP1, JP2: Bridge, Connector_PinHeader_2.54mm:PinHeader_1x02_P2.54mm_Vertical, symbol Jumper:Jumper_2_Open
- added R58: 100k, Resistor_SMD:R_0603_1608Metric_Pad0.98x0.95mm_HandSolder, symbol Device:R
- U2: LCSC (none) -> C97521
Connections:
- net +3.3V: now also R58.1
- net GND: now also D49.2 (A), JP1.1 (A), JP2.2 (B)
- net GPIO26: now also D49.1 (K), R58.2
- net RUN: now also JP1.2 (B)
- net at R9.2: now also JP2.1 (A)
Other:
- moved on the sheet: R57

Commit message: Added first draft of code
Parts:
- R5: footprint Resistor_SMD:R_0603_1608Metric_Pad0.98x0.95mm_HandSolder -> Resistor_SMD:R_0402_1005Metric; LCSC C21190 -> C11702
Changed lines of the file:
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@@
     (property "Reference" "R5" (id 0) (at 104.14 111.76 90))
     (property "Value" "1k" (id 1) (at 104.14 109.22 90))
-    (property "Footprint" "Resistor_SMD:R_0603_1608Metric_Pad0.98x0.95mm_HandSolder" (id 2) (at 104.14 110.998 90)
+    (property "Footprint" "Resistor_SMD:R_0402_1005Metric" (id 2) (at 104.14 110.998 90)
       (effects (font (size 1.27 1.27)) hide)
     )
@@
       (effects (font (size 1.27 1.27)) hide)
     )
-    (property "LCSC" "C21190" (id 4) (at 104.14 109.22 90)
+    (property "LCSC" "C11702" (id 4) (at 104.14 109.22 90)
       (effects (font (size 1.27 1.27)) hide)
     )
@@
     )
     (path "/2e3c981d-e30e-4416-8684-62698250799d"
-      (reference "R5") (unit 1) (value "1k") (footprint "Resistor_SMD:R_0603_1608Metric_Pad0.98x0.95mm_HandSolder")
+      (reference "R5") (unit 1) (value "1k") (footprint "Resistor_SMD:R_0402_1005Metric")
     )
     (path "/b4b98d32-5c21-40da-badd-2b42dabbaee3"
